File: zynthian_controller_epdf/Zynth-encoder_power_display_fan.sch (KiCad schematic (older format))
At the start: 42 parts, among them J3 40HAT, Q1 DMG2305UX, Q2 DMMT5401, Q3 Q_NMOS_GDS, U2 CAT24C32, U3 MCP23017_SS

Commit message: Submit to MFG
Parts:
- R19: LCSC C25217 -> C8218
Changed lines of the file:
@@
 F 1 "200" V 6120 5680 50  0000 C CNN
 F 2 "Resistor_SMD:R_0603_1608Metric" V 6050 5680 50  0001 C CNN
-F 3 "https://datasheet.lcsc.com/szlcsc/1811081715_UNI-ROYAL-Uniroyal-Elec-0603WAJ0201T5E_C25217.pdf" H 6120 5680 50  0001 C CNN
-F 4 "C25217" H 6120 5680 50  0001 C CNN "LCSC"
+F 3 "https://datasheet.lcsc.com/szlcsc/Uniroyal-Elec-0603WAF2000T5E_C8218.pdf" H 6120 5680 50  0001 C CNN
+F 4 "C8218" H 6120 5680 50  0001 C CNN "LCSC"
 	1    6120 5680
 	0    1    1    0
