File: Zynaptik_v2/zynthian_zynaptik.sch (KiCad schematic (older format))
At the start: 37 parts, among them U1 74LS14, U2 ADS1115IDGSR, U3 MCP4728

Commit message: Update latest PCB designs.
Parts:
- C1, C2, C3, C4, C6: symbol zynthian_zynaptik-rescue:C-device -> zynthian_zynaptik-rescue:C-device-zynthian_zynaptik-rescue
- D1, D2: symbol zynthian_zynaptik-rescue:D-device -> zynthian_zynaptik-rescue:D-device-zynthian_zynaptik-rescue
- JP1, JP2: symbol zynthian_zynaptik-rescue:Jumper_NO_Small-device -> zynthian_zynaptik-rescue:Jumper_NO_Small-device-zynthian_zynaptik-rescue
- MCP23017: symbol zynthian_zynaptik-rescue:MCP23017-microchip -> zynthian_zynaptik-rescue:MCP23017-microchip-zynthian_zynaptik-rescue
- MIDI-1, MIDI-2, MIDI-3: symbol zynthian_zynaptik-rescue:CONN_01X04_MALE-conn -> zynthian_zynaptik-rescue:CONN_01X04_MALE-conn-zynthian_zynaptik-rescue
- OC1: symbol zynthian_zynaptik-rescue:H11L1-opto -> zynthian_zynaptik-rescue:H11L1-opto-zynthian_zynaptik-rescue
- R1, R10, R2, R3, R4, R5, R6, R7, R8, R9: symbol zynthian_zynaptik-rescue:R-device -> zynthian_zynaptik-rescue:R-device-zynthian_zynaptik-rescue
- RBPi-1, Zynaptik-1: symbol zynthian_zynaptik-rescue:CONN_02X20-conn -> zynthian_zynaptik-rescue:CONN_02X20-conn-zynthian_zynaptik-rescue
