File: ZynAuCon/ZynAudioCon.kicad_pcb (KiCad board)
At the start: 2 copper layers, 56 x 74 mm, 11 parts, among them J1 Conn_02x10_Odd_Even

Commit message: Update ZynAuCon design files (v1.4)
Parts:
- moved RV1 0.50 mm to (95.8, 60.2)
- moved PHONE1 0.15 mm to (85.2, 57.4)
Routing:
- net PHONE-L: track 13.7 -> 14.4 mm
- net PHONE-R: track 27.5 -> 28.0 mm
- net GND: vias 0 -> 4
Other:
- board text added: "zynaucon v1.4"
- board text removed: "zynaucon v1.3"
Changed lines of the file:
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@@
-(kicad_pcb (version 20171130) (host pcbnew 5.1.7-a382d34a8~88~ubuntu18.04.1)
+(kicad_pcb (version 20171130) (host pcbnew 5.0.2-5.fc29)
   (general
     (thickness 1.6)
     (drawings 10)
-    (tracks 116)
+    (tracks 126)
     (zones 0)
     (modules 11)
@@
     (zone_45_only no)
     (trace_min 0.2)
+    (segment_width 0.2)
+    (edge_width 0.05)
     (via_size 0.8)
     (via_drill 0.4)
@@
     (uvia_min_size 0.2)
     (uvia_min_drill 0.1)
-    (edge_width 0.05)
-    (segment_width 0.2)
     (pcb_text_width 0.3)
     (pcb_text_size 1.5 1.5)
@@
     (pad_drill 0.762)
     (pad_to_mask_clearance 0)
+    (solder_mask_min_width 0.25)
     (aux_axis_origin 0 0)
     (visible_elements FFFFFF7F)
@@
   )
   (module ZynAudio:conn_minijack (layer F.Cu)
-    (at 85.4 57.4 180)
+    (at 85.25 57.4 180)
     (fp_text reference PHONE1 (at -3.3 -4.2) (layer F.SilkS)
       (effects (font (size 1 1) (thickness 0.15)))
@@
     (fp_line (start 3.81 8.382) (end -3.81 8.382) (layer F.SilkS) (width 0.15))
     (fp_line (start 3.81 4.826) (end 3.81 8.382) (layer F.SilkS) (width 0.15))
-    (fp_text user "3.5mm stereo phone jack" (at 0 2.794 180) (layer F.Fab)
+    (fp_text user "3.5mm stereo phone jack" (at 0 2.794 180) (layer F.Fab) hide
       (effects (font (size 0.6 0.6) (thickness 0.1)))
     )
@@
   )
   (module ZynAudio:Potentiometer_B103_5pin (layer F.Cu)
-    (at 95.8 59.7 90)
+    (at 95.758 60.198 90)
     (descr "Through hole angled pin header, 1x05, 2.00mm pitch, 4.2mm pin length, single row")
     (tags "Through hole angled pin header THT 1x05 2.00mm single row")
@@
   )
   (gr_line (start 112.16 51.89) (end 112.16 119.89) (layer Edge.Cuts) (width 0.1))
-  (gr_text "zynaucon v1.3" (at 99.5 121.4) (layer F.SilkS)
+  (gr_text "zynaucon v1.4" (at 99.5 121.4) (layer F.SilkS)
     (effects (font (size 1.15 1.15) (thickness 0.13)))
   )
@@
   (segment (start 79.902999 53.897001) (end 84.004999 53.897001) (width 0.5) (layer F.Cu) (net 2))
   (segment (start 73.66 67.82) (end 75.610001 65.869999) (width 0.5) (layer F.Cu) (net 2))
+  (via (at 85.09 60.96) (size 0.8) (drill 0.4) (layers F.Cu B.Cu) (net 2))
+  (via (at 88.646 60.96) (size 0.8) (drill 0.4) (layers F.Cu B.Cu) (net 2))
+  (via (at 70.612 56.642) (size 0.8) (drill 0.4) (layers F.Cu B.Cu) (net 2))
+  (via (at 92.964 59.182) (size 0.8) (drill 0.4) (layers F.Cu B.Cu) (net 2))
   (segment (start 96.9 102.49005) (end 73.66 79.25005) (width 0.4) (layer F.Cu) (net 3))
   (segment (start 96.9 111.339998) (end 96.9 102.49005) (width 0.4) (layer F.Cu) (net 3))
@@
   (segment (start 58.1 54.7) (end 61.2 51.6) (width 0.4) (layer B.Cu) (net 10))
   (segment (start 80.558978 54.75798) (end 92.85798 54.75798) (width 0.4) (layer B.Cu) (net 10))
-  (segment (start 98.724999 60.775001) (end 99.8 59.7) (width 0.4) (layer B.Cu) (net 11))
-  (segment (start 94.804999 60.775001) (end 98.724999 60.775001) (width 0.4) (layer B.Cu) (net 11))
-  (segment (start 94.724999 60.695001) (end 94.804999 60.775001) (width 0.4) (layer B.Cu) (net 11))
-  (segment (start 94.724999 59.154863) (end 94.724999 60.695001) (width 0.4) (layer B.Cu) (net 11))
-  (segment (start 90.928126 55.35799) (end 94.724999 59.154863) (width 0.4) (layer B.Cu) (net 11))
+  (segment (start 99.083001 60.872999) (end 99.758 60.198) (width 0.4) (layer B.Cu) (net 11))
+  (segment (start 94.488 60.998002) (end 94.762999 61.273001) (width 0.4) (layer B.Cu) (net 11))
+  (segment (start 94.488 58.928) (end 94.488 60.998002) (width 0.4) (layer B.Cu) (net 11))
+  (segment (start 91.67501 56.11501) (end 94.488 58.928) (width 0.4) (layer B.Cu) (net 11))
+  (segment (start 90.928126 55.35799) (end 91.67501 56.104874) (width 0.4) (layer B.Cu) (net 11))
+  (segment (start 91.67501 56.104874) (end 91.67501 56.11501) (width 0.4) (layer B.Cu) (net 11))
+  (segment (start 67.31 102.82) (end 64.1 99.61) (width 0.4) (layer B.Cu) (net 11))
+  (segment (start 64.1 99.61) (end 64.1 54.1) (width 0.4) (layer B.Cu) (net 11))
+  (segment (start 64.1 54.1) (end 64.6 53.6) (width 0.4) (layer B.Cu) (net 11))
+  (segment (start 94.762999 61.273001) (end 98.682999 61.273001) (width 0.4) (layer B.Cu) (net 11))
+  (segment (start 64.6 53.6) (end 78.2 53.6) (width 0.4) (layer B.Cu) (net 11))
+  (segment (start 78.2 53.6) (end 79.95799 55.35799) (width 0.4) (layer B.Cu) (net 11))
+  (segment (start 98.682999 61.273001) (end 99.083001 60.872999) (width 0.4) (layer B.Cu) (net 11))
   (segment (start 79.95799 55.35799) (end 90.928126 55.35799) (width 0.4) (layer B.Cu) (net 11))
-  (segment (start 78.2 53.6) (end 79.95799 55.35799) (width 0.4) (layer B.Cu) (net 11))
-  (segment (start 64.6 53.6) (end 78.2 53.6) (width 0.4) (layer B.Cu) (net 11))
-  (segment (start 64.1 54.1) (end 64.6 53.6) (width 0.4) (layer B.Cu) (net 11))
-  (segment (start 64.1 99.61) (end 64.1 54.1) (width 0.4) (layer B.Cu) (net 11))
-  (segment (start 67.31 102.82) (end 64.1 99.61) (width 0.4) (layer B.Cu) (net 11))
   (segment (start 106.36 115.03) (end 106.36 112.49) (width 0.5) (layer F.Cu) (net 18) (status 30))
-  (segment (start 94.26701 61.37501) (end 90.4 57.508) (width 0.4) (layer B.Cu) (net 21))
-  (segment (start 100.12499 61.37501) (end 94.26701 61.37501) (width 0.4) (layer B.Cu) (net 21))
-  (segment (start 101.8 59.7) (end 100.12499 61.37501) (width 0.4) (layer B.Cu) (net 21))
-  (segment (start 82.717019 61.975019) (end 80.4 59.658) (width 0.4) (layer B.Cu) (net 22))
-  (segment (start 80.4 59.658) (end 80.4 57.508) (width 0.4) (layer B.Cu) (net 22))
-  (segment (start 101.524981 61.975019) (end 82.717019 61.975019) (width 0.4) (layer B.Cu) (net 22))
-  (segment (start 103.8 59.7) (end 101.524981 61.975019) (width 0.4) (layer B.Cu) (net 22))
+  (segment (start 101.083001 60.872999) (end 101.758 60.198) (width 0.4) (layer B.Cu) (net 21))
+  (segment (start 100.082989 61.873011) (end 101.083001 60.872999) (width 0.4) (layer B.Cu) (net 21))
+  (segment (start 90.4 58.383) (end 93.890011 61.873011) (width 0.4) (layer B.Cu) (net 21))
+  (segment (start 93.890011 61.873011) (end 100.082989 61.873011) (width 0.4) (layer B.Cu) (net 21))
+  (segment (start 90.4 57.508) (end 90.4 58.383) (width 0.4) (layer B.Cu) (net 21))
+  (segment (start 103.083001 60.872999) (end 103.758 60.198) (width 0.4) (layer B.Cu) (net 22))
+  (segment (start 100.964 62.992) (end 103.083001 60.872999) (width 0.4) (layer B.Cu) (net 22))
+  (segment (start 83.734 62.992) (end 100.964 62.992) (width 0.4) (layer B.Cu) (net 22))
+  (segment (start 80.4 59.658) (end 83.734 62.992) (width 0.4) (layer B.Cu) (net 22))
+  (segment (start 80.4 57.508) (end 80.4 59.658) (width 0.4) (layer B.Cu) (net 22))
   (zone (net 2) (net_name GND) (layer B.Cu) (hatch edge 0.508)
     (connect_pads (clearance 0.508))
