File: ZynADAC/zynthiandac.kicad_pcb (KiCad board)
At the start: 2 copper layers, 64 x 55 mm, 77 parts, among them J1 Conn_2x20, J2 Conn_02x10_Odd_Even, J3 AudioJack2_Ground_Switch, J4 AudioJack2_Ground, J5 AudioJack2_Ground, J6 Conn_2x20, U1 PCM1863DBT, U2 AT24CS01-STUM, U3 ncp163, U4 ncp163, U5 ncp163, U6 PCM5242RHBR, X1 22.5792Mhz, X2 24.576Mhz

Commit message: Update latest PCB designs.
Routing:
- net GND: vias 51 -> 52
- net 5v: vias 2 -> 3
