File: zynthian_controller_single2_smd/zynthian_controller_single2_smd_sh.kicad_pcb (KiCad board)
At the start: 2 copper layers, 15.2 x 24.9 mm, 5 parts, among them J1 CONN_01X04, SW1 Rotary_Encoder_Switch

Commit message: Update zynthian_controller_single2_smd productionfiles (???)
Routing:
- net CON-4: vias 2 -> 3
Changed lines of the file:
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@@
     (thickness 1.6)
     (drawings 11)
-    (tracks 74)
+    (tracks 75)
     (zones 0)
     (modules 5)
@@
     (visible_elements FFFFFF7F)
     (pcbplotparams
-      (layerselection 0x310fc_ffffffff)
+      (layerselection 0x010fc_ffffffff)
       (usegerberextensions false)
       (usegerberattributes false)
@@
   (gr_line (start 164.084 94.996) (end 164.084 119.888) (angle 90) (layer Edge.Cuts) (width 0.15))
   (gr_line (start 148.844 94.996) (end 164.084 94.996) (angle 90) (layer Edge.Cuts) (width 0.15))
+  (via (at 162.60064 96.7105) (size 0.6) (drill 0.4) (layers F.Cu B.Cu) (net 4))
   (segment (start 158.924 111.1758) (end 158.877 111.125) (width 0.25) (layer B.Cu) (net 1) (status 80000))
   (segment (start 158.877 111.125) (end 158.877 112.522) (width 0.25) (layer B.Cu) (net 1) (status 80000))
