File: Zynaptik_v1/zynthian_zynaptik.kicad_pcb (KiCad board)
At the start: 2 copper layers, 119.4 x 30.5 mm, 34 parts, among them U1 74LS14

Commit message: Re-organize zynaptik subprojects & files.
Other:
- net class Default removed
