File: Zynaptik_v3/zynthian_zynaptik.kicad_pcb (KiCad board)
At the start: 2 copper layers, 119.4 x 30.5 mm, 49 parts, among them U1 74LS14, U2 ADS1115IDGSR, U3 MCP4728

Commit message: Re-organize zynaptik subprojects & files.
Other:
- net class Default removed
